File: carrier/carrier.kicad_pcb (KiCad board)
At the start: 2 copper layers, 43 parts, among them J1 Connector, J2 Connector, J3 WeAct_1, J4 WeAct_2, J5 Seansor_Header_A, J6 Seansor_Header_B, U1 TPS54302, U2 SN65HVD230, U3 ATECC608B-SSHDA

Commit message: Add files via upload
Parts:
- J5, J6: moved to B.Cu
- moved R13 127.9 mm to (227.6, 71.5)
- moved R14 125.5 mm to (225.1, 82.0)
- moved R12 123.6 mm to (223.1, 64.0)
- moved D9 113.3 mm to (207.1, 47.5)
- moved D7 111.7 mm to (206.6, 62.5)
- moved D8 110.7 mm to (205.6, 55.5)
- moved D6 108.4 mm to (202.6, 41.5)
- moved R11 105.4 mm to (205.1, 67.7)
- moved R9 104.4 mm to (199.0, 86.0)
- moved R10 97.0 mm to (191.9, 85.5)
- moved U3 94.6 mm to (172.7, 20.3), turned to 180 degrees
- moved C9 93.8 mm to (175.8, 66.5)
- moved J3 93.8 mm to (146.6, 31.3)
- moved J4 93.8 mm to (153.7, 31.3)
- moved J5 93.8 mm to (160.8, 31.3), turned to 180 degrees
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Routing:
- net CAN_H: track 0.00 -> 47.7 mm
- net GND: track 0.00 -> 45.8 mm
- net CAN_L: track 0.00 -> 45.3 mm
- net Net-(U1-SW): track 0.00 -> 36.5 mm, vias 0 -> 8
- net +12V: track 0.00 -> 27.6 mm
- net Net-(J1-Pin_1): track 0.00 -> 26.6 mm
- net +3.3V: track 0.00 -> 16.8 mm
- net CAN_TX: track 0.00 -> 6.08 mm
- net Net-(JP1-A): track 0.00 -> 5.33 mm
- net Net-(U2-Rs): track 0.00 -> 4.62 mm
- added copper zone on F.Cu, net +3.3V
- added copper zone on F.Cu, net GND
- added copper zone on F.Cu, net Net-(U1-SW)
- added copper zone on F.Cu, net Net-(U1-VIN)

Commit message: Add files via upload
Parts:
- J3, J4: footprint Connector_PinSocket_2.54mm:PinSocket_2x15_P2.54mm_Vertical -> Connector_PinSocket_2.54mm:PinSocket_2x15_P2.54mm_Vertical_SMD
- J5: footprint Connector_PinSocket_2.54mm:PinSocket_2x12_P2.54mm_Vertical -> Connector_PinSocket_2.54mm:PinSocket_2x12_P2.54mm_Vertical_SMD
- J6: footprint Connector_PinSocket_2.54mm:PinSocket_2x08_P2.54mm_Vertical -> Connector_PinSocket_2.54mm:PinSocket_2x08_P2.54mm_Vertical_SMD
- moved J6 97.5 mm to (88.9, 43.0), turned to 0 degrees
- moved R1 82.3 mm to (95.7, 54.9), turned to -90 degrees
- moved R2 80.8 mm to (91.4, 55.9), turned to 180 degrees
- moved R9 70.8 mm to (153.5, 31.7), turned to -90 degrees
- moved R10 69.2 mm to (148.4, 31.7), turned to -90 degrees
- moved C9 53.0 mm to (142.0, 25.7), turned to 180 degrees
- moved U3 33.1 mm to (142.1, 32.7), turned to 0 degrees
- moved R5 30.0 mm to (107.0, 45.7), turned to 180 degrees
- moved J5 29.9 mm to (133.3, 43.0), turned to 0 degrees
- moved R3 29.3 mm to (112.7, 55.9), turned to 180 degrees
- moved C3 28.3 mm to (106.7, 54.9), turned to 90 degrees
- moved U1 27.1 mm to (101.0, 54.9), turned to -90 degrees
- moved J4 26.4 mm to (130.1, 43.0), turned to 180 degrees
- moved C6 23.4 mm to (112.7, 50.8), turned to 180 degrees
- moved R4 20.1 mm to (112.7, 45.7), turned to 180 degrees
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Routing:
- net ADC_2: track 0.00 -> 108.4 mm, vias 0 -> 2
- net ADC_1: track 0.00 -> 100.2 mm, vias 0 -> 2
- net +3.3V: track 16.8 -> 74.5 mm
- net CAN_RX: track 0.00 -> 57.6 mm, vias 0 -> 2
- net CAN_TX: track 6.08 -> 47.7 mm, vias 0 -> 2
- net SP1_CS1: track 0.00 -> 35.3 mm, vias 0 -> 2
- net SPI2_SCK: track 0.00 -> 31.3 mm, vias 0 -> 2
- net Net-(U1-SW): track 36.5 -> 5.77 mm, vias 8 -> 7
- net PWM_4: track 0.00 -> 30.7 mm, vias 0 -> 2
- net PWM_3: track 0.00 -> 30.6 mm, vias 0 -> 2
- net +12V: track 27.6 -> 0.17 mm
- net Net-(U1-FB): track 0.00 -> 27.2 mm
- net OW_DATA: track 0.00 -> 23.5 mm, vias 0 -> 2
- net I2C2_SCL: track 0.00 -> 19.7 mm
- net SPI2_MISO: track 0.00 -> 17.7 mm, vias 0 -> 2
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- added copper zone on F.Cu, net +12V
- added copper zone on B.Cu, net Net-(U1-SW)

Commit message: Add files via upload
Parts:
- J1, J2: footprint Connector_Molex:Molex_Micro-Fit_3.0_43650-0400_1x04_P3.00mm_Horizontal -> Connector_Molex:Molex_Micro-Fit_3.0_43045-0400_2x02_P3.00mm_Horizontal
- moved R12 136.9 mm to (90.8, 28.9), turned to 90 degrees
- moved R11 124.3 mm to (87.0, 28.9), turned to 90 degrees
- moved D7 122.3 mm to (90.4, 24.2), turned to -90 degrees
- moved D6 117.9 mm to (86.0, 24.2), turned to -90 degrees
- moved R14 89.8 mm to (139.1, 56.0), turned to -90 degrees
- moved R13 84.8 mm to (144.2, 56.0), turned to -90 degrees
- moved D9 69.5 mm to (139.1, 62.3), turned to 90 degrees
- moved J6 64.4 mm to (153.2, 39.1), turned to 180 degrees
- moved D8 61.7 mm to (144.2, 62.3), turned to 90 degrees
- moved C6 17.1 mm to (101.3, 63.5)
- moved R4 15.3 mm to (106.3, 59.7)
- moved R5 15.1 mm to (101.3, 59.7), turned to 0 degrees
- moved C1 14.6 mm to (92.1, 57.3), turned to -90 degrees
- moved C4 11.5 mm to (101.1, 47.6), turned to 0 degrees
- moved L1 11.4 mm to (96.7, 28.6)
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Routing:
- net ADC_2: track 108.4 -> 7.88 mm, vias 2 -> 1
- net ADC_1: track 100.2 -> 5.85 mm, vias 2 -> 1
- net +3.3V: track 74.5 -> 152.3 mm, vias 0 -> 3
- net I2C1_SDA: track 12.7 -> 62.6 mm, vias 1 -> 2
- net Net-(U1-VIN): track 0.00 -> 39.4 mm
- net GND: track 46.2 -> 82.6 mm, vias 0 -> 292
- net Net-(U1-SW): track 5.77 -> 32.3 mm, vias 7 -> 17
- net +12V: track 0.17 -> 26.4 mm
- net SPI_CS2: track 0.00 -> 24.9 mm, vias 0 -> 1
- net I2C1_SCL: track 3.14 -> 27.0 mm, vias 2 -> 1
- net PWM_1: track 4.41 -> 24.3 mm, vias 2 -> 1
- net LED_Status: track 0.00 -> 18.9 mm
- net GPIO_4: track 9.90 -> 28.2 mm, vias 3 -> 1
- net PWM_2: track 6.28 -> 24.3 mm, vias 2 -> 1
- net PWM_4: track 30.7 -> 47.6 mm, vias 2 -> 1
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- added copper zone on B.Cu, net GND
- removed copper zone on F.Cu, net Net-(U1-VIN)
Other:
- board outline added: 104.9 x 47 mm
- copper layers 2 -> 4

Commit message: Add files via upload
Parts:
- added G***: LOGO, LOGO, F.Cu at (82.0, 64.5)
- C1: footprint Capacitor_SMD:CP_Elec_4x5.8 -> Capacitor_SMD:C_0805_2012Metric
- C4, C5: footprint Capacitor_SMD:CP_Elec_6.3x7.7 -> Capacitor_SMD:C_0805_2012Metric
- C7: footprint Capacitor_SMD:CP_Elec_4x5.4 -> Capacitor_SMD:C_0805_2012Metric
- D6: value LED -> 12V
- D7: value LED -> 3.3V
- D8: value LED -> CAN
- D9: value LED -> Status
- moved L1 11.3 mm to (96.8, 39.9)
- moved C5 5.95 mm to (100.6, 44.6)
- moved C1 1.94 mm to (92.1, 55.3)
- moved C4 1.60 mm to (100.6, 49.1)
Routing:
- net +3.3V: track 152.3 -> 167.3 mm
- net Net-(U1-SW): track 32.3 -> 20.8 mm
- net Net-(U1-VIN): track 39.4 -> 36.1 mm
- net GND: track 82.6 -> 83.5 mm, vias 292 -> 293
Other:
- copper layers 4 -> 2
- board text added: "E0001 V0.0.01"
- board text added: "SN:"
