File: store/E0001-000001.kicad_sch (KiCad schematic)
At the start: 43 parts, among them J1 Connector, J2 Connector, J3 WeAct_1, J4 WeAct_2, J5 Seansor_Header_A, J6 Seansor_Header_B, U1 TPS54302, U2 SN65HVD230, U3 ATECC608B-SSHDA

Commit message: feat(store): add E0002 KiCad project; update E0001 schematic
Add new E0002 board project (pro/sch/pcb/prl) and apply schematic
updates to E0001. Ignore KiCad *.lck editor lock files.

Signed-off-by: IIchukissII <133657307+IIchukissII@users.noreply.github.com>
Other:
- title: (none) -> carrier board
Changed lines of the file:
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@@
 	(generator_version "10.0")
 	(paper "A4")
+	(title_block
+		(title "carrier board")
+		(rev "000001")
+	)
 	(rectangle
 		(start 12.7 78.74)
