File: store/E0001-000002.kicad_pcb (KiCad board)
At the start: 2 copper layers, 104.9 x 47 mm, 45 parts, among them J1 Connector, J2 Connector, J3 WeAct_1, J4 WeAct_2, J5 Seansor_Header_A, J6 Seansor_Header_B, U1 TPS54302, U2 SN65HVD230, U3 ATECC608B-SSHDA

Commit message: hardware(E0001): release carrier v0.0.2, supersede v0.0.1 sources
Complete the v0.0.2 relayout that corrects the mirrored WeAct socket
footprint (the v0.0.1 layout defect, archived as BLOCKED). Finalize the
000002 PCB layout and the weact footprint fix.

Reissue the full design face set under E0001-000002:
- -L.csv (BOM) and -D-pinmap.md, byte-identical carry-forward from 000001
- -D.png render of the corrected layout
(the schematic and project faces already carried the 000002 identity scaffold)

Archive the remaining loose v0.0.1 sources (schematic, project files, BOM,
pin map) as E0001-000001-SUPERSEDED.zip and git rm the loose objects;
firmware -F.* stays loose (independent axis, ADR-0017 d16).

REGISTRY: add the SUPERSEDED row, update the kept-loose note to past tense,
and record the reissue policy (full face set reissued per version; one
object per identifier, ADR-0017 d15).

Fabrication outputs (gerbers, drill, -D-pos) follow in a separate commit
once exported from KiCad.

Signed-off-by: IIchukissII <133657307+IIchukissII@users.noreply.github.com>
Parts:
- renumbered J3 to IC1
Routing:
- net GPIO_3: track 0.00 -> 47.0 mm, vias 0 -> 1
- net ADC_2: track 0.00 -> 42.1 mm, vias 0 -> 1
- net +3.3V: track 154.0 -> 195.9 mm
- net SPI2_MISO: track 0.00 -> 28.7 mm, vias 0 -> 1
- net GND: track 43.1 -> 69.1 mm, vias 125 -> 246
- net PWM_3: track 0.00 -> 22.0 mm, vias 0 -> 1
- net PWM_4: track 0.00 -> 20.4 mm, vias 0 -> 1
- net SPI_CS2: track 0.00 -> 10.1 mm, vias 0 -> 1
- net CAN_RX: track 126.2 -> 122.5 mm
- net SP1_CS1: track 12.1 -> 15.4 mm
- net SPI2_SCK: track 51.0 -> 52.3 mm
- net SPI2_MOSI: track 44.3 -> 45.0 mm
- added copper zone on B.Cu, net GND
