File: store/E0002-000001.kicad_pcb (KiCad board)
At the start: 2 copper layers, 104.9 x 47 mm, 20 parts, among them J6 Seansor_Header_A, J7 Seansor_Header_B, U1 SHT45-AD1F-R2, U2 BME688, U3 SCD41-D-R2, U4 TLV70018, U5 NCP114

Commit message: M01: reposition the E0002 silkscreen and set the version to V0.0.1
Moves the LOGO to 164.372252,117.160683 with the E-number and SN text above
it, and sets the version string to E0002 V0.0.1, following E0001-000002
rather than E0006-000001, which writes V00.00.01.

Adds the board dimension annotations 104.902 and 46.99 as text outside the
outline, as E0006 carries them.

DRC 0 violations, 0 unconnected. Back-side render confirms the mark and both
text lines read the right way round.

Signed-off-by: IIchukissII <133657307+IIchukissII@users.noreply.github.com>
Parts:
- moved G*** 51.4 mm to (164.4, 117.2)
Other:
- board text added: "E0002 V0.0.1"
- board text removed: "E0002 V00.00.01"
