File: store/E0001-000003.kicad_pcb (KiCad board)
At the start: 2 copper layers, 104.9 x 47 mm, 45 parts, among them IC1 WeAct_1, J1 Connector, J2 Connector, J3 WeAct_1, J4 WeAct_2, J5 Seansor_Header_A, J6 Seansor_Header_B, U1 TPS54302, U2 SN65HVD230, U3 ATECC608B-SSHDA

Commit message: store: supersede carrier v0.0.2 with E0001-000003
E0001-000003: full nine-face set reissued, PA6 routed to STRAP_1, zones refilled.
E0001-000002: nine faces archived SUPERSEDED, loose objects removed.
REGISTRY.md: fab-package row and strap-transport note moved to v0.0.3; superseded
row added.
Pin-map references retargeted in 4 specs, firmware/README.md and
E0006-000001-D-pinmap.md.

Signed-off-by: IIchukissII <133657307+IIchukissII@users.noreply.github.com>
Connections:
- J3 pad 15: unconnected-(J3-Pin_15-Pad15) -> STRAP_1
Routing:
- net STRAP_1: track 0.00 -> 39.8 mm, vias 0 -> 1
Changed lines of the file:
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@@
 			(size 3 1)
 			(layers "F.Cu" "F.Mask" "F.Paste")
-			(net "unconnected-(J3-Pin_15-Pad15)")
+			(net "STRAP_1")
 			(pinfunction "Pin_15_15")
 			(pintype "passive")
@@
 	)
 	(segment
+		(start 150.763114 36.634816)
+		(end 153.303114 34.094816)
+		(width 0.1017)
+		(layer "F.Cu")
+		(net "STRAP_1")
+	)
+	(segment
+		(start 153.303114 34.094816)
+		(end 155.998784 34.094816)
+		(width 0.1017)
+		(layer "F.Cu")
+		(net "STRAP_1")
+	)
+	(segment
+		(start 121.047677 40.968631)
+		(end 122.047677 40.968631)
+		(width 0.1017)
+		(layer "F.Cu")
+		(net "STRAP_1")
+	)
+	(segment
+		(start 145.22813 37.63485)
+		(end 146.228164 36.634816)
+		(width 0.1017)
+		(layer "F.Cu")
+		(net "STRAP_1")
+	)
+	(segment
+		(start 124.336827 37.677781)
+		(end 124.379758 37.63485)
+		(width 0.1017)
+		(layer "F.Cu")
+		(net "STRAP_1")
+	)
+	(segment
+		(start 124.379758 37.63485)
+		(end 145.22813 37.63485)
+		(width 0.1017)
+		(layer "F.Cu")
+		(net "STRAP_1")
+	)
+	(segment
+		(start 156.0068 34.0868)
+		(end 155.998784 34.094816)
+		(width 0.1017)
+		(layer "F.Cu")
+		(net "STRAP_1")
+	)
+	(segment
+		(start 122.047677 40.968631)
+		(end 124.336827 38.679481)
+		(width 0.1017)
+		(layer "F.Cu")
+		(net "STRAP_1")
+	)
+	(segment
+		(start 124.336827 38.679481)
+		(end 124.336827 37.677781)
+		(width 0.1017)
+		(layer "F.Cu")
+		(net "STRAP_1")
+	)
+	(segment
+		(start 146.228164 36.634816)
+		(end 150.763114 36.634816)
+		(width 0.1017)
+		(layer "F.Cu")
+		(net "STRAP_1")
+	)
+	(via
+		(at 156.0068 34.0868)
+		(size 0.6)
+		(drill 0.3)
+		(layers "F.Cu" "B.Cu")
+		(net "STRAP_1")
+	)
+	(segment
+		(start 155.701929 33.781929)
+		(end 156.0068 34.0868)
+		(width 0.1017)
+		(layer "B.Cu")
+		(net "STRAP_1")
+	)
+	(segment
+		(start 155.701929 32.766364)
+		(end 155.701929 33.781929)
+		(width 0.1017)
+		(layer "B.Cu")
+		(net "STRAP_1")
+	)
+	(segment
