File: store/E0001-000003.kicad_sch (KiCad schematic)
At the start: 43 parts, among them J1 Connector, J2 Connector, J3 WeAct_1, J4 WeAct_2, J5 Seansor_Header_A, J6 Seansor_Header_B, U1 TPS54302, U2 SN65HVD230, U3 ATECC608B-SSHDA

Commit message: store: supersede carrier v0.0.2 with E0001-000003
E0001-000003: full nine-face set reissued, PA6 routed to STRAP_1, zones refilled.
E0001-000002: nine faces archived SUPERSEDED, loose objects removed.
REGISTRY.md: fab-package row and strap-transport note moved to v0.0.3; superseded
row added.
Pin-map references retargeted in 4 specs, firmware/README.md and
E0006-000001-D-pinmap.md.

Signed-off-by: IIchukissII <133657307+IIchukissII@users.noreply.github.com>
Connections:
- net STRAP_1: now also J3.15 (Pin_15)
