File: store/E0003-000001.kicad_sch (KiCad schematic)
At the start: 23 parts, among them J8 Seansor_Header_A, J9 Seansor_Header_B, U1 AS7343-DLGM, U2 AS7331-AQFM, U3 TLV70018, U4 PCA9306

Commit message: store: re-annotate E0003 and complete its supply nets
E0003-000001.kicad_sch: designators re-annotated (J8/J9 to J1/J2;
U1 PCA9306, U2 TLV70018, U3 AS7331, U4 AS7343; passives renumbered).
C1/C2 10 uF, C3 4.7 uF, C7 100 nF added at the AS7343 VDD pin.
U3 VDDA/VDDD tied to +3.3V; they sat on an isolated net carrying only
R4, which ERC reported as an undriven power input.
PWR_FLAG on +3.3V, GND, GNDA and the TLV70018 input node.
ERC 0 errors, 16 isolated-label warnings on unused header signals.

Signed-off-by: IIchukissII <133657307+IIchukissII@users.noreply.github.com>
Parts:
- removed C5: 1uF, Capacitor_SMD:C_0805_2012Metric, symbol Device:C
- added C2: 10uF, Capacitor_SMD:C_0805_2012Metric, symbol Device:C
- added C3: 4.7uF, Capacitor_SMD:C_0805_2012Metric, symbol Device:C
- renumbered C4 to C1, C6 to C4, C2 to C5, C3 to C6, C1 to C7, J8 to J1, J9 to J2, R10 to R1, R5 to R10, R9 to R2, R8 to R3, R6 to R4, R7 to R5, R1 to R6, R2 to R7, R3 to R8, R4 to R9, U4 to U1, U3 to U2, U2 to U3, U1 to U4
Connections:
- net +1V8: now also C3.2
- net +3.3V: now also R4.1, U3.10 (VDDD), U3.3 (VDDA)
- net GND: now also C2.2, C3.1
- net at C1.1, FB1.2, U2.1 (IN)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: now also C2.1
Other:
- moved on the sheet: C1
